File: hardware_design/pcb/interconnect.kicad_sch (KiCad schematic)
At the start: 8 parts, among them J10 Conn_01x10_Socket, J11 Conn_01x10_Socket, J12 Conn_01x10_Pin, J13 Conn_01x10_Socket, J14 Conn_01x10_Pin, J15 Conn_01x10_Socket, J16 Conn_01x10_Pin, J9 Conn_01x10_Pin

Commit message: Rev 2 schematic & circuit board
Connections:
- net +3.3V: no longer J11.8 (Pin_8), J12.8 (Pin_8), J15.8 (Pin_8), J16.8 (Pin_8)
- net ALG_A: now also J11.8 (Pin_8); no longer J11.9 (Pin_9)
- net ALG_B: now also J11.9 (Pin_9); no longer J11.10 (Pin_10)
- net LED renamed CLOCK_OUT
- new net ALG_C: J11.10 (Pin_10)
- new net B_8: J12.8 (Pin_8)
- no-connect marks 4 -> 6
